File: 400W-Mono-ClassAB-Amplifier.kicad_pcb (KiCad board)
At the start: 0 parts

Commit message: Update to well-formed KiCad v7 schematic, PCB and project files (400W)
Parts:
- added ?: , , F.Cu at (0.00, 0.00)
- added ?: , Resistors_SMD:R_0805, F.Cu at (50.0, 50.0)
Other:
- net class default removed
Changed lines of the file:
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@@
 (kicad_pcb (version 20220614) (host pcbnew "(7.0.10)")
-  (general
-    (thickness 1.6)
+  (general (thickness 1.6))
+  (paper "A4")
+  (layers (0 "F.Cu") (31 "B.Cu") (42 "Edge.Cuts"))
+  (setup (last_trace_width 0.254) (trace_clearance 0.25) (zone_clearance 0.5) (via_size 0.8) (via_drill 0.4))
+  (net (code 1) (name "NET1"))
+  (module "Resistors_SMD:R_0805" (layer F.Cu) (at 50 50 0)
+    (pad 1 smd rect (at -1.25 0) (size 1.5 1.8) (layers F.Cu F.Paste F.Mask))
+    (pad 2 smd rect (at 1.25 0) (size 1.5 1.8) (layers F.Cu F.Paste F.Mask))
   )
-  (paper "A4")
-  (layers
-    (0 "F.Cu")
-    (31 "B.Cu")
-    (32 "B.Adhes")
-    (33 "F.Adhes")
-    (34 "F.SilkS")
-    (35 "B.SilkS")
-    (36 "F.Paste")
-    (37 "B.Paste")
-    (38 "F.Mask")
-    (39 "B.Mask")
-    (40 "Dwgs.User")
-    (41 "Cmts.User")
-    (42 "Edge.Cuts")
-    (43 "Margin")
-    (44 "Fabrication")
-  )
-  (setup (last_trace_width 0.254) (trace_clearance 0.25) (zone_clearance 0.5) (zone_45_only yes) (via_size 0.8) (via_drill 0.4) (via_min_size 0.6) (edge_width 0.15))
-  (net_class default  (clearance 0.25) (trace_width 0.254) (via_dia 0.8) (via_drill 0.4) (via_min_size 0.6) (zone_connect 0))
-  (nets
-    (net (code 1) (name "NET1"))
-  )
-  (modules
-    (module "Resistors_SMD:R_0805" (layer F.Cu)
-      (at 50 50 0)
-      (pad 1 smd rect (at -1.25 0) (size 1.5 1.8) (layers F.Cu F.Paste F.Mask))
-      (pad 2 smd rect (at 1.25 0) (size 1.5 1.8) (layers F.Cu F.Paste F.Mask))
-    )
-  )
+  (footprint "" )
   (properties (board "400W-Mono-ClassAB-Amplifier"))
 )

Commit message: Add corrected KiCad v7 project/schematic/pcb for CI (400W)
Parts:
- removed the ? at (0.00, 0.00)
Changed lines of the file:
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@@
   (setup (last_trace_width 0.254) (trace_clearance 0.25) (zone_clearance 0.5) (via_size 0.8) (via_drill 0.4))
   (net (code 1) (name "NET1"))
+  ; Minimal module using a standard KiCad footprint name
   (module "Resistors_SMD:R_0805" (layer F.Cu) (at 50 50 0)
     (pad 1 smd rect (at -1.25 0) (size 1.5 1.8) (layers F.Cu F.Paste F.Mask))
     (pad 2 smd rect (at 1.25 0) (size 1.5 1.8) (layers F.Cu F.Paste F.Mask))
   )
-  (footprint "" )
   (properties (board "400W-Mono-ClassAB-Amplifier"))
 )
