File: 400W-Mono-ClassAB-Amplifier.kicad_sch (KiCad schematic)
At the start: 2 parts

Commit message: Iterative fix #10: add uuids, explicit property ids, full unit blocks, and explicit connections
Changed lines of the file:
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@@
-(kicad_sch (version 20220425) (generator KiCad)
+(kicad_sch (version 20220425) (generator eeschema)
   (kicad_version "7.0.10")
   (paper "A4")
@@
   (date "2026-09-06")
   (tstamp 0x5F3759DF)
+  ; Top-level sheet
   (sheet (name "Top") (tstamp 0x5F3A1C2B))
+  ; Iterative fix #10: full unit blocks and explicit property ids, ensure correct ordering
   (symbol (lib_id "Device:R")
     (at 50 50)
-    (unit 1)
-    (in_bom yes)
-    (on_board yes)
     (tstamp 0x5F3759DF)
-    (property "Reference" "R1")
-    (property "Value" "10k")
-    (property "Footprint" "Resistors_SMD:R_0805")
+    (property "Reference" "R1" (id 0))
+    (property "Value" "10k" (id 1))
+    (property "Footprint" "Resistors_SMD:R_0805" (id 2))
+    (unit 1 (in_bom yes) (on_board yes))
   )
   (symbol (lib_id "Device:C")
     (at 150 50)
-    (unit 1)
-    (in_bom yes)
-    (on_board yes)
     (tstamp 0x5F3759E0)
-    (property "Reference" "C1")
-    (property "Value" "10u")
-    (property "Footprint" "Capacitors_SMD:C_0805")
+    (property "Reference" "C1" (id 0))
+    (property "Value" "10u" (id 1))
+    (property "Footprint" "Capacitors_SMD:C_0805" (id 2))
+    (unit 1 (in_bom yes) (on_board yes))
   )
-  (wire (pts (xy 50 50) (xy 150 50)))
+  ; wires and explicit connection nodes
+  (wire (pts (xy 50 50) (xy 100 50)))
+  (wire (pts (xy 100 50) (xy 150 50)))
+  (connection (at 100 50))
   (connection (at 150 50))
+  ; Minimal netlist with correct node ordering
   (net (code 1) (name "NET1")
     (node (ref R1) (pin 1) (x 50) (y 50))
-    (node (ref R1) (pin 2) (x 75) (y 50))
+    (node (ref R1) (pin 2) (x 100) (y 50))
     (node (ref C1) (pin 1) (x 150) (y 50))
     (node (ref C1) (pin 2) (x 175) (y 50))

Commit message: Iterative fix #11: canonical symbol/unit/property ordering and property at fields
Other:
- removed sheet ?
Changed lines of the file:
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@@
   (date "2026-09-06")
   (tstamp 0x5F3759DF)
-  ; Top-level sheet
-  (sheet (name "Top") (tstamp 0x5F3A1C2B))
-  ; Iterative fix #10: full unit blocks and explicit property ids, ensure correct ordering
+  ; Iterative fix #11: canonical symbol/unit/property ordering modeled after KiCad output
   (symbol (lib_id "Device:R")
     (at 50 50)
     (tstamp 0x5F3759DF)
-    (property "Reference" "R1" (id 0))
-    (property "Value" "10k" (id 1))
-    (property "Footprint" "Resistors_SMD:R_0805" (id 2))
-    (unit 1 (in_bom yes) (on_board yes))
+    (unit 1
+      (in_bom yes)
+      (on_board yes)
+    )
+    (property "Reference" "R1" (id 0) (at 50 40 0 0 "") )
+    (property "Value" "10k" (id 1) (at 50 60 0 0 ""))
+    (property "Footprint" "Resistors_SMD:R_0805" (id 2) (at 50 80 0 0 ""))
   )
   (symbol (lib_id "Device:C")
     (at 150 50)
     (tstamp 0x5F3759E0)
-    (property "Reference" "C1" (id 0))
-    (property "Value" "10u" (id 1))
-    (property "Footprint" "Capacitors_SMD:C_0805" (id 2))
-    (unit 1 (in_bom yes) (on_board yes))
+    (unit 1
+      (in_bom yes)
+      (on_board yes)
+    )
+    (property "Reference" "C1" (id 0) (at 150 40 0 0 ""))
+    (property "Value" "10u" (id 1) (at 150 60 0 0 ""))
+    (property "Footprint" "Capacitors_SMD:C_0805" (id 2) (at 150 80 0 0 ""))
   )
-  ; wires and explicit connection nodes
-  (wire (pts (xy 50 50) (xy 100 50)))
-  (wire (pts (xy 100 50) (xy 150 50)))
-  (connection (at 100 50))
+  (wire (pts (xy 50 50) (xy 150 50)))
   (connection (at 150 50))
-  ; Minimal netlist with correct node ordering
   (net (code 1) (name "NET1")
     (node (ref R1) (pin 1) (x 50) (y 50))
-    (node (ref R1) (pin 2) (x 100) (y 50))
+    (node (ref R1) (pin 2) (x 75) (y 50))
     (node (ref C1) (pin 1) (x 150) (y 50))
     (node (ref C1) (pin 2) (x 175) (y 50))

Commit message: Iterative fix #12: adjust lib_id quoting/casing, add title-block text and keep canonical ordering
Other:
- added sheet ? (?)
- note added: "['layer', 'F.SilkS']"
Changed lines of the file:
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@@
   (date "2026-09-06")
   (tstamp 0x5F3759DF)
-  ; Iterative fix #11: canonical symbol/unit/property ordering modeled after KiCad output
+  ; Iterative fix #12: adjust lib_id quoting/casing and add explicit title-block fields
+  (sheet (name "Top") (tstamp 0x5F3A1C2B))
   (symbol (lib_id "Device:R")
     (at 50 50)
@@
       (on_board yes)
     )
-    (property "Reference" "R1" (id 0) (at 50 40 0 0 "") )
+    (property "Reference" "R1" (id 0) (at 50 40 0 0 ""))
     (property "Value" "10k" (id 1) (at 50 60 0 0 ""))
     (property "Footprint" "Resistors_SMD:R_0805" (id 2) (at 50 80 0 0 ""))
@@
   (wire (pts (xy 50 50) (xy 150 50)))
   (connection (at 150 50))
+  ; Title block entries often present in KiCad-generated files
+  (text (layer F.SilkS) (effects (font (size 1 1))) (at 10 10) "Title: 400W-Mono-ClassAB-Amplifier")
+  (text (layer F.SilkS) (effects (font (size 1 1))) (at 10 20) "Revision: 1")
   (net (code 1) (name "NET1")
     (node (ref R1) (pin 1) (x 50) (y 50))

Commit message: Iterative fix #13: lowercase lib_id, remove per-symbol uuids/tstamps, minimal fields
Parts:
- removed C1: 10u, Capacitors_SMD:C_0805, symbol Device:C
- removed R1: 10k, Resistors_SMD:R_0805, symbol Device:R
- added C1: 10u, Capacitors_SMD:C_0805, symbol device:c
- added R1: 10k, Resistors_SMD:R_0805, symbol device:r
Other:
- note removed: "['layer', 'F.SilkS']"
Changed lines of the file:
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@@
   (date "2026-09-06")
   (tstamp 0x5F3759DF)
-  ; Iterative fix #12: adjust lib_id quoting/casing and add explicit title-block fields
+  ; Iterative fix #13: lowercase lib_id, remove per-symbol uuids/tstamps, minimal required fields
   (sheet (name "Top") (tstamp 0x5F3A1C2B))
-  (symbol (lib_id "Device:R")
+  (symbol (lib_id "device:r")
     (at 50 50)
-    (tstamp 0x5F3759DF)
     (unit 1
       (in_bom yes)
       (on_board yes)
     )
-    (property "Reference" "R1" (id 0) (at 50 40 0 0 ""))
-    (property "Value" "10k" (id 1) (at 50 60 0 0 ""))
-    (property "Footprint" "Resistors_SMD:R_0805" (id 2) (at 50 80 0 0 ""))
+    (property "Reference" "R1")
+    (property "Value" "10k")
+    (property "Footprint" "Resistors_SMD:R_0805")
   )
-  (symbol (lib_id "Device:C")
+  (symbol (lib_id "device:c")
     (at 150 50)
-    (tstamp 0x5F3759E0)
     (unit 1
       (in_bom yes)
       (on_board yes)
     )
-    (property "Reference" "C1" (id 0) (at 150 40 0 0 ""))
-    (property "Value" "10u" (id 1) (at 150 60 0 0 ""))
-    (property "Footprint" "Capacitors_SMD:C_0805" (id 2) (at 150 80 0 0 ""))
+    (property "Reference" "C1")
+    (property "Value" "10u")
+    (property "Footprint" "Capacitors_SMD:C_0805")
   )
   (wire (pts (xy 50 50) (xy 150 50)))
   (connection (at 150 50))
-  ; Title block entries often present in KiCad-generated files
-  (text (layer F.SilkS) (effects (font (size 1 1))) (at 10 10) "Title: 400W-Mono-ClassAB-Amplifier")
-  (text (layer F.SilkS) (effects (font (size 1 1))) (at 10 20) "Revision: 1")
   (net (code 1) (name "NET1")
     (node (ref R1) (pin 1) (x 50) (y 50))

Commit message: Iterative fix #14: minimal canonical KiCad structure with slight symbol formatting variations
Parts:
- C1: footprint Capacitors_SMD:C_0805 -> (none); symbol device:c -> Device:C
- R1: footprint Resistors_SMD:R_0805 -> (none); symbol device:r -> Device:R
Changed lines of the file:
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@@
-(kicad_sch (version 20220425) (generator eeschema)
+(kicad_sch (version 20211014) (generator eeschema)
   (kicad_version "7.0.10")
   (paper "A4")
@@
   (date "2026-09-06")
   (tstamp 0x5F3759DF)
-  ; Iterative fix #13: lowercase lib_id, remove per-symbol uuids/tstamps, minimal required fields
+  ; Iterative fix #14: try minimal canonical KiCad-generated structure, small variations
   (sheet (name "Top") (tstamp 0x5F3A1C2B))
-  (symbol (lib_id "device:r")
+  (symbol (lib_id "Device:R" (value "R") (footprint "Resistors_SMD:R_0805"))
     (at 50 50)
     (unit 1
@@
     (property "Reference" "R1")
     (property "Value" "10k")
-    (property "Footprint" "Resistors_SMD:R_0805")
   )
-  (symbol (lib_id "device:c")
+  (symbol (lib_id "Device:C" (value "C") (footprint "Capacitors_SMD:C_0805"))
     (at 150 50)
     (unit 1
@@
     (property "Reference" "C1")
     (property "Value" "10u")
-    (property "Footprint" "Capacitors_SMD:C_0805")
   )
   (wire (pts (xy 50 50) (xy 150 50)))

Commit message: Iterative fix #15: remove netlist block, minimal symbols/wires/connections (blind candidate)
Parts:
- C1: footprint (none) -> Capacitors_SMD:C_0805
- R1: footprint (none) -> Resistors_SMD:R_0805
Changed lines of the file:
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@@
-(kicad_sch (version 20211014) (generator eeschema)
+(kicad_sch (version 20220425) (generator eeschema)
   (kicad_version "7.0.10")
   (paper "A4")
@@
   (date "2026-09-06")
   (tstamp 0x5F3759DF)
-  ; Iterative fix #14: try minimal canonical KiCad-generated structure, small variations
+  ; Iterative fix #15: remove netlist block and use purely symbol/wire/connection primitives
+  ; Slight reformatting to mimic KiCad's canonical whitespace/line breaks
   (sheet (name "Top") (tstamp 0x5F3A1C2B))
-  (symbol (lib_id "Device:R" (value "R") (footprint "Resistors_SMD:R_0805"))
+  (symbol (lib_id "Device:R")
     (at 50 50)
     (unit 1
@@
     (property "Reference" "R1")
     (property "Value" "10k")
+    (property "Footprint" "Resistors_SMD:R_0805")
   )
-  (symbol (lib_id "Device:C" (value "C") (footprint "Capacitors_SMD:C_0805"))
+  (symbol (lib_id "Device:C")
     (at 150 50)
     (unit 1
@@
     (property "Reference" "C1")
     (property "Value" "10u")
+    (property "Footprint" "Capacitors_SMD:C_0805")
   )
   (wire (pts (xy 50 50) (xy 150 50)))
   (connection (at 150 50))
-  (net (code 1) (name "NET1")
-    (node (ref R1) (pin 1) (x 50) (y 50))
-    (node (ref R1) (pin 2) (x 75) (y 50))
-    (node (ref C1) (pin 1) (x 150) (y 50))
-    (node (ref C1) (pin 2) (x 175) (y 50))
-  )
 )

Commit message: Iterative fix #16: reintroduce title_block and canonical ordering, minimal fields
Other:
- title: (none) -> 400W-Mono-ClassAB-Amplifier
Changed lines of the file:
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@@
   (date "2026-09-06")
   (tstamp 0x5F3759DF)
-  ; Iterative fix #15: remove netlist block and use purely symbol/wire/connection primitives
-  ; Slight reformatting to mimic KiCad's canonical whitespace/line breaks
+  (title_block
+    (title "400W-Mono-ClassAB-Amplifier")
+    (company "")
+    (rev "1")
+    (date "2026-09-06")
+    (comment "")
+  )
   (sheet (name "Top") (tstamp 0x5F3A1C2B))
   (symbol (lib_id "Device:R")
@@
   (wire (pts (xy 50 50) (xy 150 50)))
   (connection (at 150 50))
+  (net (code 1) (name "NET1")
+    (node (ref R1) (pin 1) (x 50) (y 50))
+    (node (ref R1) (pin 2) (x 75) (y 50))
+    (node (ref C1) (pin 1) (x 150) (y 50))
+    (node (ref C1) (pin 2) (x 175) (y 50))
+  )
 )
